File: Panels/Apr25/IotRollerBlinds.kicad_pcb (KiCad board)
At the start: 2 copper layers, 135 x 78 mm, 178 parts

Commit message: Update IotRollerBlinds.kicad_pcb
Parts:
- removed JD3: 5?A@1V 90? Single 3.53V~3.67V 200mW 3.6V SOD-323 Zener Diod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, Diode_SMD:D_SOD-323
- removed JD4: Red 615~630nm 1.9~2.2V 0603 Light Emitting Diodes (LED) RoHS, LED_SMD:LED_0603_1608Metric
- removed JQ1, JQ4: 20V 3.1A 860mW 112m?@4.5V,2.8A 1V@250?A P Channel SOT-23(SO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, Package_TO_SOT_SMD:SOT-23
- removed JQ2, JQ3: 60V 115mA 200mW 7.5?@10V,500mA 2.5V@250?A N Channel SOT-23(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, Package_TO_SOT_SMD:SOT-23
- removed JR15, JR16: ±1% 1/10W Thick Film Resistors 75V ±100ppm/? -55?~+155? 10k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, Resistor_SMD:R_0603_1608Metric
- removed the REF** at (44.0, 92.0)
- removed the REF** at (104.0, 125.0)
- added BC10: drv.vm_cap1, Capacitor_SMD:CP_Elec_8x10, F.Cu at (40.0, 98.0)
- added JC10: mcu.vcc_cap1, Capacitor_SMD:C_0603_1608Metric, F.Cu at (128.5, 113.0)
- added JC11: mcu.en_pull.c, Capacitor_SMD:C_0603_1608Metric, F.Cu at (114.5, 116.0)
- added JC12: trig.cbyp, Capacitor_SMD:C_0603_1608Metric, F.Cu at (78.5, 128.0)
- added JC9: mcu.vcc_cap0, Capacitor_SMD:C_0805_2012Metric, F.Cu at (124.5, 113.0)
- added JL1: mp2722.power_path.inductor, Inductor_SMD:L_1210_3225Metric, F.Cu at (91.5, 130.0)
- added JTP4: v3v3, edg:TestPoint_TE_RCT_0805, F.Cu at (108.5, 116.0)
- added RC14: drv.vm_cap1, Capacitor_SMD:CP_Elec_8x10, F.Cu at (57.0, 65.0)
- added REF**: Indicator_IdDots_4, edg:Indicator_IdDots_4, F.Cu at (50.0, 92.0)
- added REF**: Indicator_IdDots_4, edg:Indicator_IdDots_4, B.Cu at (104.5, 125.0)
- BC1, OC1, RC1: value 50V 100nF X7R ±10% 0603 Multilayer Ceramic Capacitors MLCC - SMD/SMT ROHS -> reg_3v3.hf_in_cap
- BC2, OC2, RC2: value 50V 100nF X7R ±10% 0603 Multilayer Ceramic Capacitors MLCC - SMD/SMT ROHS -> reg_3v3.boot_cap
- BC3, RC3: value 50V 10uF X5R ±10% 1206 Multilayer Ceramic Capacitors MLCC - SMD/SMT ROHS -> reg_3v3.power_path.in_cap.c[0]
- BC4, RC4: value X5R 25V ±10% 10uF 0805 Multilayer Ceramic Capacitors MLCC - SMD/SMT ROHS -> reg_3v3.power_path.in_cap.c[1]; footprint Capacitor_SMD:C_0805_2012Metric -> Capacitor_SMD:C_1206_3216Metric
- BC5, OC4, RC5: value X5R 25V ±10% 10uF 0805 Multilayer Ceramic Capacitors MLCC - SMD/SMT ROHS -> reg_3v3.power_path.out_cap
- BC6, RC6: value 50V 100nF X7R ±10% 0603 Multilayer Ceramic Capacitors MLCC - SMD/SMT ROHS -> mcu.vcc_cap0; footprint Capacitor_SMD:C_0603_1608Metric -> Capacitor_SMD:C_0805_2012Metric
- BC7, RC7: value 50V 1uF X5R ±10% 0603 Multilayer Ceramic Capacitors MLCC - SMD/SMT ROHS -> mcu.vcc_cap1
- BC8, RC8: value 50V 100nF X7R ±10% 0603 Multilayer Ceramic Capacitors MLCC - SMD/SMT ROHS -> mcu.en_pull.c
- BC9, RC13: value -40?~+105? 2000hrs@105? 47uF 5.4mm 35V 6.3mm ±20% SMD,6.3x5.4mm Aluminum Electrolytic Capacitors - SMD ROHS -> drv.vm_cap0; footprint Capacitor_SMD:CP_Elec_3x5.4 -> Capacitor_SMD:C_0603_1608Metric
- BD1, OD1, RD1: value 5?A@1V 90? Single 3.53V~3.67V 200mW 3.6V SOD-323 Zener Diodes ROHS -> prot_3v3
- BD2, OD2, RD2: value Red 615~630nm 1.9~2.2V 0603 Light Emitting Diodes (LED) RoHS -> ledr.package
- BF1, RF1: value 01550900M -> fuse
- BFB1, RFB1: value 700mA 1 200m? 30?@100MHz ±25% 0603 Ferrite Beads ROHS -> ferrite
- BH1, JH1, OH1, RH1: value (none) -> jlc_th.th1
- BH2, JH2, OH2, RH2: value (none) -> jlc_th.th2
- BH3, JH3, OH3, RH3: value (none) -> jlc_th.th3
- BJ1, RJ1: value B2B-PH-K -> pwr
- BJ2, RJ2: value B2B-PH-K -> pwr_out
- BJ3: value B6B-XH-A -> conn
- BJ4, JJ3, OJ1, RJ3: value (none) -> mcu.prog
- BJ5, RJ4: value SM04B-SRSS-TB -> qwiic
- BL1, RL1: value 620mA 22uH ±10% 270m? 1210 Inductors (SMD) ROHS -> reg_3v3.power_path.inductor; footprint Inductor_SMD:L_1210_3225Metric -> Inductor_SMD:L_Sunlord_SWPA4030S
- BR1, OR1, RR1: value ±1% 1/10W Thick Film Resistors 75V ±100ppm/? -55?~+155? 6.8k? 0603 Chip Resistor - Surface Mount ROHS -> reg_3v3.fb.top_res
- BR10, RR11: value ±1% 1/4W Thick Film Resistors 200V ±800ppm/? -55?~+155? 680m? 1206 Chip Resistor - Surface Mount ROHS -> drv.isen_res
- BR2, OR2, RR2: value ±1% 1/10W Thick Film Resistors 75V ±100ppm/? -55?~+155? 1.5k? 0603 Chip Resistor - Surface Mount ROHS -> reg_3v3.fb.bottom_res
- BR3, OR3, RR3: value ±1% 1/10W Thick Film Resistors 75V ±100ppm/? -55?~+155? 510k? 0603 Chip Resistor - Surface Mount ROHS -> reg_3v3.en_res
- BR4, JR3, OR4, RR4: value ±1% 1/10W Thick Film Resistors 75V ±100ppm/? -55?~+155? 10k? 0603 Chip Resistor - Surface Mount ROHS -> mcu.en_pull.r
- BR5, OR5, RR5: value ±1% 1/10W Thick Film Resistors 75V ±100ppm/? -55?~+155? 1k? 0603 Chip Resistor - Surface Mount ROHS -> ledr.res
- BR6, RR6: value ±1% 1/10W Thick Film Resistors 75V ±100ppm/? -55?~+155? 56k? 0603 Chip Resistor - Surface Mount ROHS -> vin_sense.top_res
- BR7, RR7: value ±1% 1/10W Thick Film Resistors 75V ±100ppm/? -55?~+155? 10k? 0603 Chip Resistor - Surface Mount ROHS -> vin_sense.bottom_res
- BR8: value ±1% 1/10W Thick Film Resistors 75V ±100ppm/? -55?~+155? 4.7k? 0603 Chip Resistor - Surface Mount ROHS -> qwiic_pull.scl_res
- BR9: value ±1% 1/10W Thick Film Resistors 75V ±100ppm/? -55?~+155? 4.7k? 0603 Chip Resistor - Surface Mount ROHS -> qwiic_pull.sda_res
- BU1, OU2, RU1: value TPS54202H -> reg_3v3.ic
- BU2, JU3, OU3, RU2: value ESP32-C3-WROOM-02 -> mcu.ic
- BU3, RU6: value DRV8870DDAR -> drv.ic
- JC1: value 50V 1uF X5R ±10% 0603 Multilayer Ceramic Capacitors MLCC - SMD/SMT ROHS -> mp2722.vbst_cap
- JC2: value 50V 1uF X5R ±10% 0603 Multilayer Ceramic Capacitors MLCC - SMD/SMT ROHS -> mp2722.pmid_cap; footprint Capacitor_SMD:C_0603_1608Metric -> Capacitor_SMD:C_0805_2012Metric
- JC3: value 25V 4.7uF X5R ±10% 0805 Multilayer Ceramic Capacitors MLCC - SMD/SMT ROHS -> mp2722.batt_cap; footprint Capacitor_SMD:C_0805_2012Metric -> Capacitor_SMD:C_1206_3216Metric
- JC4: value 25V 4.7uF X5R ±10% 0805 Multilayer Ceramic Capacitors MLCC - SMD/SMT ROHS -> mp2722.vcc_cap
- JC5: value X5R 25V ±10% 10uF 0805 Multilayer Ceramic Capacitors MLCC - SMD/SMT ROHS -> mp2722.power_path.in_cap
- JC6: value 50V 100nF X7R ±10% 0603 Multilayer Ceramic Capacitors MLCC - SMD/SMT ROHS -> mp2722.power_path.out_cap; footprint Capacitor_SMD:C_0603_1608Metric -> Capacitor_SMD:C_0805_2012Metric
- JC7: value 50V 1uF X5R ±10% 0603 Multilayer Ceramic Capacitors MLCC - SMD/SMT ROHS -> reg_3v3.in_cap
- JC8: value 50V 100nF X7R ±10% 0603 Multilayer Ceramic Capacitors MLCC - SMD/SMT ROHS -> reg_3v3.out_cap
- JD1: value 30V 370mV@1mA 30mA SOD-323 Schottky Barrier Diodes (SBD) ROHS -> prot_3v3
- JD2: value 30V 370mV@1mA 30mA SOD-323 Schottky Barrier Diodes (SBD) ROHS -> ledr.package; footprint Diode_SMD:D_SOD-323 -> LED_SMD:LED_0603_1608Metric
- JJ1: value B2B-PH-K -> bat
- JJ2: value COM-15111 -> usb
- JR1: value ±1% 1/10W Thick Film Resistors 75V ±100ppm/? -55?~+155? 5.1k? 0603 Chip Resistor - Surface Mount ROHS -> fake_ntc.top_res
- JR10: value ±1% 1/10W Thick Film Resistors 75V ±100ppm/? -55?~+155? 10k? 0603 Chip Resistor - Surface Mount ROHS -> ledr.res
- JR11: value ±1% 1/10W Thick Film Resistors 75V ±100ppm/? -55?~+155? 10k? 0603 Chip Resistor - Surface Mount ROHS -> vbat_sense.top_res
- JR12: value ±1% 1/10W Thick Film Resistors 75V ±100ppm/? -55?~+155? 10k? 0603 Chip Resistor - Surface Mount ROHS -> vbat_sense.bottom_res
- JR13: value ±1% 1/10W Thick Film Resistors 75V ±100ppm/? -55?~+155? 10k? 0603 Chip Resistor - Surface Mount ROHS -> i2c_pull.scl_res
- JR14: value ±1% 1/10W Thick Film Resistors 75V ±100ppm/? -55?~+155? 1k? 0603 Chip Resistor - Surface Mount ROHS -> i2c_pull.sda_res
- JR2: value ±1% 1/10W Thick Film Resistors 75V ±100ppm/? -55?~+155? 5.1k? 0603 Chip Resistor - Surface Mount ROHS -> fake_ntc.bottom_res
- JR4: value ±1% 1/10W Thick Film Resistors 75V ±100ppm/? -55?~+155? 10k? 0603 Chip Resistor - Surface Mount ROHS -> ax1_div.top_res
- JR5: value ±1% 1/10W Thick Film Resistors 75V ±100ppm/? -55?~+155? 10k? 0603 Chip Resistor - Surface Mount ROHS -> ax1_div.bottom_res
- JR6: value ±1% 1/10W Thick Film Resistors 75V ±100ppm/? -55?~+155? 4.99k? 0603 Chip Resistor - Surface Mount ROHS -> ax2_div.top_res
- JR7: value ±1% 1/10W Thick Film Resistors 75V ±100ppm/? -55?~+155? 10k? 0603 Chip Resistor - Surface Mount ROHS -> ax2_div.bottom_res
- JR8: value ±1% 1/10W Thick Film Resistors 75V ±100ppm/? -55?~+155? 10k? 0603 Chip Resistor - Surface Mount ROHS -> trig_div.top_res
- JR9: value ±1% 1/10W Thick Film Resistors 75V ±100ppm/? -55?~+155? 10k? 0603 Chip Resistor - Surface Mount ROHS -> trig_div.bottom_res
- JSW1: value 3.9x2.9mm Switch -> mcu.boot
- JSW2: value 3.9x2.9mm Switch -> sw[0]
- JSW3: value 3.9x2.9mm Switch -> sw[1]
- JSW4: value 3.9x2.9mm Switch -> sw[2]
- JTP2: value gnd -> vusb
- JTP3: value v3v3 -> gnd
- JU1: value AP7215-33YG-13 -> mp2722.ic; footprint Package_TO_SOT_SMD:SOT-89-3 -> edg:MPS_QFN-22_2.5x3.5mm_P0.4mm
- JU2: value MCP73831T-2ACI/OT -> reg_3v3.ic; footprint Package_TO_SOT_SMD:SOT-23-5 -> Package_TO_SOT_SMD:SOT-89-3
- JU4: value (none) -> stick
- JU5: value A1304ELHLX-T -> trig.ic
- OC3: value 25V 22uF X5R ±10% 1206 Multilayer Ceramic Capacitors MLCC - SMD/SMT ROHS -> reg_3v3.power_path.in_cap
- OC5: value X5R 25V ±10% 10uF 0805 Multilayer Ceramic Capacitors MLCC - SMD/SMT ROHS -> mcu.vcc_cap0
- OC6: value 50V 100nF X7R ±10% 0603 Multilayer Ceramic Capacitors MLCC - SMD/SMT ROHS -> mcu.vcc_cap1
- OC7: value 50V 1uF X5R ±10% 0603 Multilayer Ceramic Capacitors MLCC - SMD/SMT ROHS -> mcu.en_pull.c
- OC8: value 50V 100nF X7R ±10% 0603 Multilayer Ceramic Capacitors MLCC - SMD/SMT ROHS -> can.vdd_cap
- OD3: value 20mA 285mcd 3.3V 518nm Colorless transparence -40?~+85? 520nm~535nm Emerald 120° 110mW 0603 Light Emitting Diodes (LED)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 -> ledg.package
- OD4: value White 0603 Light Emitting Diodes (LED) RoHS -> ledw.package
- OFB1: value 200mA 1 450m? 600?@100MHz ±25% 0603 Ferrite Beads ROHS -> ferrite
- OL1: value 620mA 22uH ±10% 270m? 1210 Inductors (SMD) ROHS -> reg_3v3.power_path.inductor
- OR6: value ±1% 1/10W Thick Film Resistors 75V ±100ppm/? -55?~+155? 1k? 0603 Chip Resistor - Surface Mount ROHS -> ledg.res
- OR7: value ±1% 1/10W Thick Film Resistors 75V ±100ppm/? -55?~+155? 1k? 0603 Chip Resistor - Surface Mount ROHS -> ledw.res
- OR8: value ±1% 1/10W Thick Film Resistors 75V ±100ppm/? -55?~+155? 91k? 0603 Chip Resistor - Surface Mount ROHS -> vobd_sense.top_res
- OR9: value ±1% 1/10W Thick Film Resistors 75V ±100ppm/? -55?~+155? 10k? 0603 Chip Resistor - Surface Mount ROHS -> vobd_sense.bottom_res
- OU1: value (none) -> obd
- OU4: value SN65HVD230DR -> can.ic
- RC10: value 50V 100nF X7R ±10% 0603 Multilayer Ceramic Capacitors MLCC - SMD/SMT ROHS -> encb.cin
- RC11: value 50V 1uF X5R ±10% 0603 Multilayer Ceramic Capacitors MLCC - SMD/SMT ROHS -> als.vcc_cap
- RC12: value 50V 100nF X7R ±10% 0603 Multilayer Ceramic Capacitors MLCC - SMD/SMT ROHS -> als.dvi_cap
- RC9: value 50V 100nF X7R ±10% 0603 Multilayer Ceramic Capacitors MLCC - SMD/SMT ROHS -> enca.cin
- RJ5: value 533980271 -> motor
- RR10: value ±1% 1/10W Thick Film Resistors 75V ±100ppm/? -55?~+155? 1k? 0603 Chip Resistor - Surface Mount ROHS -> als.dvi_res
- RR8: value ±1% 1/10W Thick Film Resistors 75V ±100ppm/? -55?~+155? 4.7k? 0603 Chip Resistor - Surface Mount ROHS -> i2c_pull.scl_res
- RR9: value ±1% 1/10W Thick Film Resistors 75V ±100ppm/? -55?~+155? 4.7k? 0603 Chip Resistor - Surface Mount ROHS -> i2c_pull.sda_res
- RSW1: value 5.1mm switch -> sw
- RU3: value AH1806-W-7 -> enca.ic
- RU4: value AH1806-W-7 -> encb.ic
- RU5: value BH1750 -> als.ic
- moved BC8 78.8 mm to (126.0, 91.0), turned to 180 degrees
- moved RC5 55.5 mm to (44.0, 86.0)
- moved BC5 54.6 mm to (72.0, 101.0)
- moved RC8 53.8 mm to (82.0, 62.0)
- moved JC5 42.1 mm to (85.5, 130.0), turned to -90 degrees
- moved JC6 36.2 mm to (93.5, 124.0)
- moved JTP3 34.9 mm to (77.5, 133.0)
- moved JR5 32.8 mm to (114.5, 118.0)
- moved JR3 29.6 mm to (114.5, 114.0)
- moved JC8 29.1 mm to (104.5, 116.0), turned to 0 degrees
- moved JR2 28.9 mm to (101.5, 127.0)
- moved JR1 28.7 mm to (101.5, 125.0)
- moved JR6 27.8 mm to (110.5, 127.0), turned to 0 degrees
- moved JR4 25.2 mm to (110.5, 118.0)
- moved JR13 21.9 mm to (94.5, 115.0), turned to -90 degrees
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Connections:
- BC4 pad 1: Bv3v3 -> Bvin
- BC7 pad 1: Bmcu.program_en_node -> Bv3v3
- BC8 pad 1: Bvin -> Bmcu.program_en_node
- JC1 pad 1: Jgate.pwr_out -> Jmp2722.vbst_cap.pos
- JC1 pad 2: Jgnd -> Jmp2722.vbst_cap.neg
- JC2 pad 1: Jv3v3 -> Jmp2722.ic.pmid
- JC3 pad 1: Jusb.pwr -> Jvbat
- JC4 pad 1: Jvbat -> Jmp2722.ic.vcc
- JC5 pad 1: Jv3v3 -> Jvusb
- JC6 pad 1: Jv3v3 -> Jmp2722.pwr_out
- JC7 pad 1: Jmcu.program_en_node -> Jmp2722.pwr_out
- JD1 pad 1: Jstick.sw -> Jv3v3
- JD1 pad 2: Jgate.pull_res.b -> Jgnd
- JD2 pad 1: Jstick.sw -> Jledr.res.a
- JD2 pad 2: Jgate.btn_out -> Jv3v3
- JJ2 pad A4: Jusb.pwr -> Jvusb
- JJ2 pad A5: Jusb.conn.cc.cc1 -> Jmp2722.cc.cc1
- JJ2 pad A9: Jusb.pwr -> Jvusb
- JJ2 pad B4: Jusb.pwr -> Jvusb
- JJ2 pad B5: Jusb.conn.cc.cc2 -> Jmp2722.cc.cc2
- JJ2 pad B9: Jusb.pwr -> Jvusb
- JR1 pad 1: Jgnd -> Jmp2722.vrntc
- JR1 pad 2: Jusb.conn.cc.cc1 -> Jfake_ntc.output
- JR10 pad 1: Jstick.ax2 -> Jledr.res.a
- JR10 pad 2: Jax2_div.output -> Jmcu.program_boot_node
- JR11 pad 1: Jax2_div.output -> Jvbat
- JR11 pad 2: Jgnd -> Jvbat_sense.output
- JR12 pad 1: Jtrig.out -> Jvbat_sense.output
- JR12 pad 2: Jtrig_div.output -> Jgnd
- JR13 pad 1: Jtrig_div.output -> Jv3v3
- JR13 pad 2: Jgnd -> Ji2c_pull.i2c.scl
- JR14 pad 1: Jledr.res.a -> Jv3v3
- JR14 pad 2: Jmcu.program_boot_node -> Ji2c_pull.i2c.sda
- JR2 pad 1: Jgnd -> Jfake_ntc.output
- JR2 pad 2: Jusb.conn.cc.cc2 -> Jgnd
- JR3 pad 1: Jvbat -> Jv3v3
- JR3 pad 2: Jgate.pull_res.b -> Jmcu.program_en_node
- JR4 pad 1: Jgnd -> Jstick.ax1
- JR4 pad 2: Jgate.control -> Jax1_div.output
- JR5 pad 1: Jvbat -> Jax1_div.output
- JR5 pad 2: Jvbat_sense_gate.pre.drain -> Jgnd
- JR6 pad 1: Jchg.prog_res.a -> Jstick.ax2
- JR6 pad 2: Jgnd -> Jax2_div.output
- JR7 pad 1: Jv3v3 -> Jax2_div.output
- JR7 pad 2: Jmcu.program_en_node -> Jgnd
- JR8 pad 1: Jstick.ax1 -> Jtrig.out
- JR8 pad 2: Jax1_div.output -> Jtrig_div.output
- JR9 pad 1: Jax1_div.output -> Jtrig_div.output
- JTP2 pad 1: Jgnd -> Jvusb
- JTP3 pad 1: Jv3v3 -> Jgnd
- JU1 pad 1: Jgnd -> Jmp2722.cc.cc1
- JU1 pad 2: Jgate.pwr_out -> Jvusb
- JU1 pad 3: Jv3v3 -> Jmp2722.ic.pmid
- JU2 pad 1: Jchg.stat -> Jgnd
- JU2 pad 2: Jgnd -> Jmp2722.pwr_out
- JU2 pad 3: Jvbat -> Jv3v3
- JU3 pad 14: Jvbat_sense_gate.control -> Ji2c_pull.i2c.sda
- JU3 pad 4: Jgate.btn_out -> Ji2c_pull.i2c.scl
- JU3 pad 5: Jgate.control -> Jstick.sw
- RC11 pad 1: Rals.dvi_res.b -> Rv3v3
- RC12 pad 1: Rvin -> Rals.dvi_res.b
- RC4 pad 1: Rv3v3 -> Rvin
- RC7 pad 1: Rmcu.program_en_node -> Rv3v3
- RC8 pad 1: Rv3v3 -> Rmcu.program_en_node
Routing:
- net Ji2c_pull.i2c.sda: track 0.00 -> 54.5 mm, vias 0 -> 4
- net Ji2c_pull.i2c.scl: track 0.00 -> 52.6 mm, vias 0 -> 2
- net Jgate.control: track 43.8 -> 0.00 mm
- net Jvbat_sense_gate.control: track 43.4 -> 0.00 mm, vias 2 -> 0
- net Jgate.btn_out: track 39.2 -> 0.00 mm
- net Jstick.sw: track 22.5 -> 56.2 mm
- net Jvbat_sense_gate.output: track 26.3 -> 0.00 mm
- net Jmp2722.pwr_out: track 0.00 -> 21.0 mm, vias 0 -> 7
- net Jgate.pwr_out: track 20.9 -> 0.00 mm, vias 2 -> 0
- net Jvusb: track 0.00 -> 20.6 mm, vias 0 -> 4
- net Jusb.pwr: track 16.9 -> 0.00 mm, vias 1 -> 0
- net Jv3v3: track 152.3 -> 168.4 mm, vias 7 -> 6
- net Jfake_ntc.output: track 0.00 -> 15.6 mm, vias 0 -> 2
- net Jmp2722.cc.cc1: track 0.00 -> 12.8 mm, vias 0 -> 1
- net Jmp2722.cc.cc2: track 0.00 -> 12.4 mm, vias 0 -> 1
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- added copper zone on F.Cu, net Jmp2722.ic.pmid
- added copper zone on F.Cu, net Jmp2722.pwr_out
- added copper zone on F.Cu, net Jmp2722.vbst_cap.neg
- added copper zone on F.Cu, net Jvbat
- added copper zone on B.Cu, net Jvusb
- added copper zone on F.Cu, net Jvusb
- removed copper zone on B.Cu, net Jusb.pwr
Other:
- board size 135 x 78 mm -> 134.5 x 78 mm
- board text added: "131.4mm length 125.3mm length to hat 5.8mm length of hat 19.8mm W 17.5mm W hat 27.0 L hat edge to notch edge inner 0.8mm notch depth 2.5mm notch width"
- board text added: "Left (-x) toward motor 81.1mm top L Notches at (from battery side) 16.2mm, 60.2mm 4.3mmW, 2.2mmD 83.0mm bot L Notches at 26.2mm, 70.2mm 28.1mm W 27.7mm (base), 26.6mm (top) D roller ~1mm clearance from board edge to roller ~55mm L to switch center ~72mm L to ALS center"

Commit message: wip fabdata
Parts:
- added LANT1: mcu.ant, Diode_SMD:D_1206_3216Metric, F.Cu at (114.1, 56.2)
- added LC1: reg_3v3.hf_in_cap, Capacitor_SMD:C_0402_1005Metric, F.Cu at (148.0, 63.5)
- added LC10: mcu.vddspi_cap, Capacitor_SMD:C_0402_1005Metric, F.Cu at (136.0, 52.0)
- added LC11: mcu.pi.c1, Capacitor_SMD:C_0603_1608Metric, F.Cu at (120.9, 48.8)
- added LC12: mcu.pi.c2, Capacitor_SMD:C_0603_1608Metric, F.Cu at (117.0, 51.8)
- added LC13: mcu.vdd3p3_l_cap, Capacitor_SMD:C_0402_1005Metric, F.Cu at (123.5, 50.0)
- added LC14: mcu.vdd3p3_cap, Capacitor_SMD:C_0402_1005Metric, F.Cu at (126.0, 49.0)
- added LC15: mcu.crystal.cap_a, Capacitor_SMD:C_0402_1005Metric, F.Cu at (128.8, 46.0)
- added LC16: mcu.crystal.cap_b, Capacitor_SMD:C_0402_1005Metric, F.Cu at (133.2, 46.0)
- added LC17: mcu.en_pull.c, Capacitor_SMD:C_0402_1005Metric, F.Cu at (126.0, 53.0)
- added LC18: tof.vdd_cap[0], Capacitor_SMD:C_0402_1005Metric, F.Cu at (141.6, 59.6)
- added LC19: tof.vdd_cap[1], Capacitor_SMD:C_0805_2012Metric, F.Cu at (142.5, 62.3)
- added LC2: reg_3v3.boot_cap, Capacitor_SMD:C_0402_1005Metric, F.Cu at (144.0, 70.0)
- added LC20: led_drv[0].cap, Capacitor_SMD:C_0402_1005Metric, F.Cu at (113.0, 63.0)
- added LC21: led_drv[0].boot_cap, Capacitor_SMD:C_0402_1005Metric, F.Cu at (115.5, 68.5)
- added LC22: led_drv[0].power_path.in_cap, Capacitor_SMD:C_0805_2012Metric, F.Cu at (115.5, 63.0)
- added LC23: led_drv[0].power_path.out_cap, Capacitor_SMD:C_1206_3216Metric, F.Cu at (111.0, 63.5)
- added LC24: led_drv[1].cap, Capacitor_SMD:C_0402_1005Metric, F.Cu at (116.2, 76.6)
- added LC25: led_drv[1].boot_cap, Capacitor_SMD:C_0402_1005Metric, F.Cu at (121.8, 78.7)
- added LC26: led_drv[1].power_path.in_cap, Capacitor_SMD:C_0805_2012Metric, F.Cu at (117.9, 74.8)
- added LC27: led_drv[1].power_path.out_cap, Capacitor_SMD:C_1206_3216Metric, F.Cu at (115.1, 78.4)
- added LC28: led_drv[2].cap, Capacitor_SMD:C_0402_1005Metric, F.Cu at (128.0, 84.0)
- added LC29: led_drv[2].boot_cap, Capacitor_SMD:C_0402_1005Metric, F.Cu at (133.5, 81.5)
- added LC3: reg_3v3.power_path.in_cap, Capacitor_SMD:C_1206_3216Metric, F.Cu at (151.0, 65.0)
- added LC30: led_drv[2].power_path.in_cap, Capacitor_SMD:C_0805_2012Metric, F.Cu at (128.0, 81.5)
- added LC31: led_drv[2].power_path.out_cap, Capacitor_SMD:C_1206_3216Metric, F.Cu at (128.5, 86.0)
- added LC32: led_drv[3].cap, Capacitor_SMD:C_0402_1005Metric, F.Cu at (141.6, 80.8)
- added LC33: led_drv[3].boot_cap, Capacitor_SMD:C_0402_1005Metric, F.Cu at (143.7, 75.2)
- added LC34: led_drv[3].power_path.in_cap, Capacitor_SMD:C_0805_2012Metric, F.Cu at (139.8, 79.1)
- added LC35: led_drv[3].power_path.out_cap, Capacitor_SMD:C_1206_3216Metric, F.Cu at (143.4, 81.9)
- added LC4: reg_3v3.power_path.out_cap, Capacitor_SMD:C_1206_3216Metric, F.Cu at (151.0, 70.0)
- added LC5: mcu.vdd_bulk_cap, Capacitor_SMD:C_0805_2012Metric, F.Cu at (121.0, 56.0)
- added LC6: mcu.vdda_cap0, Capacitor_SMD:C_0402_1005Metric, F.Cu at (126.8, 46.0)
- added LC7: mcu.vdda_cap1, Capacitor_SMD:C_0402_1005Metric, F.Cu at (127.8, 46.0)
- added LC8: mcu.vddrtc_cap, Capacitor_SMD:C_0402_1005Metric, F.Cu at (126.0, 54.0)
- added LC9: mcu.vddcpu_cap, Capacitor_SMD:C_0402_1005Metric, F.Cu at (136.0, 53.0)
- added LD1: prot_3v3, Diode_SMD:D_SOD-323, F.Cu at (119.5, 54.5)
- added LD2: ledr.package, LED_SMD:LED_0603_1608Metric, F.Cu at (139.0, 74.0)
- added LH1: jlc_th.th1, edg:JlcToolingHole_1.152mm, F.Cu at (125.1, 80.3)
- added LH2: jlc_th.th2, edg:JlcToolingHole_1.152mm, F.Cu at (149.5, 73.7)
- added LH3: jlc_th.th3, edg:JlcToolingHole_1.152mm, F.Cu at (118.2, 49.5)
- added LJ1: pwr, Connector_JST:JST_SH_SM02B-SRSS-TB_1x02-1MP_P1.00mm_Horizontal, F.Cu at (146.7, 59.5)
- added LJ2: mcu.prog, Connector:Tag-Connect_TC2030-IDC-NL_2x03_P1.27mm_Vertical, F.Cu at (138.5, 48.0)
- added LJ3: qwiic, Connector_JST:JST_SH_SM04B-SRSS-TB_1x04-1MP_P1.00mm_Horizontal, F.Cu at (143.0, 54.0)
- added LL1: reg_3v3.power_path.inductor, Inductor_SMD:L_1210_3225Metric, F.Cu at (147.0, 70.0)
- added LL2: mcu.pi.l, Inductor_SMD:L_0603_1608Metric, F.Cu at (119.4, 50.9)
- added LL3: mcu.vdd3p3_l, Inductor_SMD:L_0402_1005Metric, F.Cu at (126.0, 50.0)
- added LL4: led_drv[0].power_path.inductor, Inductor_SMD:L_1210_3225Metric, F.Cu at (111.5, 68.5)
- added LL5: led_drv[1].power_path.inductor, Inductor_SMD:L_1210_3225Metric, F.Cu at (119.0, 81.6)
- added LL6: led_drv[2].power_path.inductor, Inductor_SMD:L_1210_3225Metric, F.Cu at (133.5, 85.5)
- added LL7: led_drv[3].power_path.inductor, Inductor_SMD:L_1210_3225Metric, F.Cu at (146.6, 78.0)
- added LR1: reg_3v3.fb.top_res, Resistor_SMD:R_0603_1608Metric, F.Cu at (144.0, 66.0)
- added LR10: qwiic_pull.sda_res, Resistor_SMD:R_0402_1005Metric, F.Cu at (139.8, 50.8)
- added LR11: tof_pull.scl_res, Resistor_SMD:R_0402_1005Metric, F.Cu at (137.4, 55.4)
- added LR12: tof_pull.sda_res, Resistor_SMD:R_0402_1005Metric, F.Cu at (136.7, 54.7)
- added LR13: led_drv[0].rsense, Resistor_SMD:R_0603_1608Metric, F.Cu at (115.5, 70.0)
- added LR14: led_drv[1].rsense, Resistor_SMD:R_0603_1608Metric, F.Cu at (122.9, 79.8)
- added LR15: led_drv[2].rsense, Resistor_SMD:R_0603_1608Metric, F.Cu at (135.0, 81.5)
- added LR16: led_drv[3].rsense, Resistor_SMD:R_0603_1608Metric, F.Cu at (144.8, 74.1)
- added LR2: reg_3v3.fb.bottom_res, Resistor_SMD:R_0603_1608Metric, F.Cu at (142.5, 66.0)
- added LR3: reg_3v3.en_res, Resistor_SMD:R_0402_1005Metric, F.Cu at (146.0, 63.5)
- added LR4: mcu.en_pull.r, Resistor_SMD:R_0402_1005Metric, F.Cu at (126.0, 52.0)
- added LR5: ledr.res, Resistor_SMD:R_0402_1005Metric, F.Cu at (137.0, 76.0)
- added LR6: v12_sense.top_res, Resistor_SMD:R_0603_1608Metric, F.Cu at (119.8, 59.8)
- added LR7: v12_sense.bottom_res, Resistor_SMD:R_0603_1608Metric, F.Cu at (118.5, 58.5)
- added LR8: qwiic_pwr_res, Resistor_SMD:R_0402_1005Metric, F.Cu at (142.3, 60.3)
- added LR9: qwiic_pull.scl_res, Resistor_SMD:R_0402_1005Metric, F.Cu at (138.4, 52.2)
- added LTP1: v12, edg:TestPoint_TE_RCT_0805, F.Cu at (138.3, 83.6)
- added LTP2: gnd, edg:TestPoint_TE_RCT_0805, F.Cu at (123.7, 83.6)
- added LTP3: v3v3, edg:TestPoint_TE_RCT_0805, F.Cu at (113.4, 73.3)
- added LU1: reg_3v3.ic, Package_TO_SOT_SMD:SOT-23-6, F.Cu at (147.0, 66.0)
- added LU2: mcu.ic, Package_DFN_QFN:QFN-32-1EP_5x5mm_P0.5mm_EP3.65x3.65mm, F.Cu at (131.0, 51.0)
- added LU3: tof.ic, OptoDevice:ST_VL53L0X, F.Cu at (139.5, 57.5)
- added LU4: led_drv[0].ic, Package_TO_SOT_SMD:SOT-23-6, F.Cu at (115.5, 66.0)
- added LU5: led_drv[1].ic, Package_TO_SOT_SMD:SOT-23-6, F.Cu at (120.0, 77.0)
- added LU6: led_drv[2].ic, Package_TO_SOT_SMD:SOT-23-6, F.Cu at (131.0, 81.5)
- added LU7: led_drv[3].ic, Package_TO_SOT_SMD:SOT-23-6, F.Cu at (142.0, 77.0)
- added LX1: mcu.crystal.package, Crystal:Crystal_SMD_2520-4Pin_2.5x2.0mm, F.Cu at (131.0, 45.8)
- added REF**: MouseBites, edg:HalfMouseBites_Recessed, F.Cu at (131.0, 89.0)
- added REF**: MouseBites, edg:HalfMouseBites_Recessed, F.Cu at (108.0, 66.0)
- added REF**: MouseBites, edg:HalfMouseBites_Recessed, F.Cu at (108.2, 66.0)
- added REF**: MouseBites, edg:HalfMouseBites_Recessed, F.Cu at (131.0, 88.8)
- added UU4: Duck, edg:Symbol_Duckling, B.Cu at (114.0, 67.5)
Routing:
- net Lv3v3: track 0.00 -> 111.1 mm, vias 0 -> 20
- net Lmcu.program_boot_node: track 0.00 -> 47.8 mm, vias 0 -> 3
- net Lled_drv[3].pwm: track 0.00 -> 46.3 mm, vias 0 -> 2
- net Lled_drv[2].pwm: track 0.00 -> 38.2 mm, vias 0 -> 2
- net Lled_drv[1].pwm: track 0.00 -> 30.8 mm, vias 0 -> 2
- net Lled_drv[0].pwm: track 0.00 -> 23.5 mm, vias 0 -> 2
- net Lv12: track 0.00 -> 22.5 mm, vias 0 -> 17
- net Lqwiic_pwr_res.pwr_out: track 0.00 -> 21.9 mm, vias 0 -> 2
- net Lv12_sense.output: track 0.00 -> 16.2 mm
- net Lmcu.program_en_node: track 0.00 -> 15.8 mm, vias 0 -> 2
- net Lqwiic_i2c.sda: track 0.00 -> 15.2 mm
- net Ltof_pull.i2c.scl: track 0.00 -> 14.7 mm, vias 0 -> 2
- net Ltof_pull.i2c.sda: track 0.00 -> 13.2 mm, vias 0 -> 2
- net Lqwiic_i2c.scl: track 0.00 -> 10.8 mm
- net Lmcu.program_uart_node.a_tx: track 0.00 -> 10.7 mm, vias 0 -> 2
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- added copper zone on B.Cu, net Lgnd
- added copper zone on F.Cu, net Lgnd
- added copper zone on F.Cu, net Lled_drv[0].boot_cap.neg
- added copper zone on F.Cu, net Lled_drv[0].leda
- added copper zone on F.Cu, net Lled_drv[1].boot_cap.neg
- added copper zone on F.Cu, net Lled_drv[1].leda
- added copper zone on F.Cu, net Lled_drv[2].boot_cap.neg
- added copper zone on F.Cu, net Lled_drv[2].leda
- added copper zone on F.Cu, net Lled_drv[3].boot_cap.neg
- added copper zone on F.Cu, net Lled_drv[3].leda
- added copper zone on F.Cu, net Lreg_3v3.boot_cap.neg
- added copper zone on B.Cu, net Lv12
- added copper zone on F.Cu, net Lv12
- added copper zone on B.Cu, net Lv3v3
- added copper zone on F.Cu, net Lv3v3
Other:
- board size 134.5 x 78 mm -> 134.5 x 94 mm
